Commit message: new file:   urdf.rviz 	modified:   urdf/assembly_hamster.urdf

File: urdf/assembly_hamster.urdf (robot description, URDF)
Before this commit: robot assembly_hamster, 11 links, 10 joints
Joints:
- joint joint_1: origin xyz=0 0 0.0202 rpy=1.5708 0 0 -> xyz=0 0 0 rpy=1.5708 0 0

Commit message: gitignore

File: urdf/assembly_hamster.urdf (robot description, URDF)
Before this commit: robot assembly_hamster, 11 links, 10 joints
Joints:
- joint joint_2_31: axis 1 0 0 -> 0 0 0; type continuous -> fixed
- joint joint_3_base: axis 0 0 0 -> 1 0 0
- joint joint_end_effector: origin xyz=0 0.032 -0.045 rpy=1.5708 0.021754 3.1416 -> xyz=0 0.032 -0.045 rpy=1.5708 0 3.1416

Commit message: last

File: urdf/assembly_hamster.urdf (robot description, URDF)
Before this commit: robot assembly_hamster, 11 links, 10 joints
Links:
- removed link 2_2_Link
- removed link 2_31_Link
- removed link 2_3_Link
- removed link 3_2_Link
Joints:
- removed joint joint_2_2
- removed joint joint_2_3
- removed joint joint_2_31
- removed joint joint_3_2
- joint joint_2_1: origin xyz=-0.0285 0.055 0 rpy=1.5708 0 -1.3472 -> xyz=-0.0285 0.055 0 rpy=1.5708 0 -1.5708
- joint joint_3_1: origin xyz=-0.048498 0.3244 0 rpy=0 0 2.1095 -> xyz=-0.048498 0.3244 0 rpy=0 0 1.8008
- joint joint_last: axis 0 0 0 -> 1 0 0; origin xyz=0 0.25 -0.0005 rpy=2.1095 -1.5708 0 -> xyz=0 0.25 -0.0005 rpy=3.14 -1.57 -1.5708; type fixed -> continuous

Commit message: add mimic

File: urdf/assembly_hamster.urdf (robot description, URDF)
Before this commit: robot assembly_hamster, 7 links, 6 joints
Joints:
- joint joint_last: mimic (none) -> joint=joint_3_1 multiplier=-1 offset=0

Commit message: add 2 mimic joint

File: urdf/assembly_hamster.urdf (robot description, URDF)
Before this commit: robot assembly_hamster, 7 links, 6 joints
Links:
- added link last_Link_2
Joints:
- added joint joint_last_2: type continuous, parent 3_1_Link, child last_Link_2, origin xyz=0 0.25 -0.0005 rpy=3.14 -1.57 -1.5708, axis 1 0 0, mimic joint=joint_2_1 multiplier=-1 offset=0
- joint joint_last: origin xyz=0 0.25 -0.0005 rpy=3.14 -1.57 -1.5708 -> xyz=0 0 0 rpy=0 0 0; parent 3_1_Link -> last_Link_2
