Commit message: to xacro

File: urdf/assembly_hamster.xacro (robot description, xacro)
@@ -73,5 +73,5 @@
   <joint
     name="joint_1"
-    type="continuous">
+    type="revolute">
     <origin
       xyz="0 0 0.0202"
@@ -83,4 +83,9 @@
     <axis
       xyz="0 1 0" />
+      <limit
+      lower="3"
+      upper="-3"
+      effort="1000.0"
+      velocity="0.1" />
   </joint>
   <link
@@ -126,5 +131,5 @@
   <joint
     name="joint_2_1"
-    type="continuous">
+    type="revolute">
     <origin
       xyz="-0.0285 0.055 0"
@@ -136,4 +141,9 @@
     <axis
       xyz="0 1 0" />
+      <limit
+      lower="1.5"
+      upper="-0.8"
+      effort="1000.0"
+      velocity="0.1" />
   </joint>
   <link
@@ -232,5 +242,5 @@
   <joint
     name="joint_3_1"
-    type="continuous">
+    type="revolute">
     <origin
       xyz="-0.048498 0.3244 0"
@@ -242,4 +252,9 @@
     <axis
       xyz="0 0 1" />
+      <limit
+      lower="1.3"
+      upper="-3"
+      effort="1000.0"
+      velocity="0.1" />
   </joint>
   <link
@@ -288,5 +303,5 @@
   <joint
     name="joint_last_2"
-    type="continuous">
+    type="revolute">
     <origin
       xyz="0 0.25 -0.0005"
@@ -299,8 +314,13 @@
       xyz="1 0 0" />
        <mimic joint="joint_2_1"  multiplier="-1" offset="0" />
+  <limit
+      lower="3"
+      upper="-3"
+      effort="1000.0"
+      velocity="0.1" />
   </joint>
   <joint
     name="joint_last"
-    type="continuous">
+    type="revolute">
     <origin
        xyz="0 0 0"
@@ -313,7 +333,33 @@
       xyz="1 0 0" />
        <mimic joint="joint_3_1"  multiplier="-1" offset="0" />
-  </joint>
-  <link
-    name="end_Link">
+  <limit
+      lower="3"
+      upper="-3"
+      effort="1000.0"
+      velocity="0.1" />
+  </joint>
+<link
+name="end_link">
+</link>
+<joint
+    name="joint_gripper"
+    type="revolute">
+    <origin
+      xyz="0 0.032 -0.045"
+      rpy="1.5708 0 3.1416" />
+    <parent
+      link="last_Link" />
+    <child
+      link="end_link" />
+    <axis
+      xyz="0 0 1" />
+      <limit
+      lower="3.14"
+      upper="-3.14"
+      effort="1000.0"
+      velocity="0.1" />
+  </joint>
+  <link
+    name="gripper">
     <inertial>
       <origin
@@ -356,14 +402,17 @@
   <joint
     name="joint_end_effector"
-    type="continuous">
-    <origin
-      xyz="0 0.032 -0.045"
-      rpy="1.5708 0 3.1416" />
-    <parent
-      link="last_Link" />
-    <child
-      link="end_Link" />
-    <axis
-      xyz="0 0 1" />
-  </joint>
+    type="fixed">
+    <origin
+      xyz="0 0 0"
+      rpy="0 0 0" />
+    <parent
+      link="end_link" />
+    <child
+      link="gripper" />
+  </joint>
+      <gazebo>
+        <plugin name="gazebo_ros_control" filename="libgazebo_ros_control.so">
+        <robotNamespace>/rrr_arm</robotNamespace>
+        </plugin>
+    </gazebo>
 </robot>
